Commit message: Add mixed real + mock hardware example

File: zenoh_host/wbot_description/urdf/wbot_macro.xacro (robot description, xacro)
@@ -10,5 +10,5 @@
     <xacro:include filename="$(find turtlebot3_description)/urdf/turtlebot3_waffle.urdf"/>
     <xacro:include filename="$(find wbot_description)/urdf/wbot.ros2_control.xacro"/>
-    <xacro:property name="ros2_control_name" value="wbot_control"/>
+    <xacro:property name="ros2_control_name" value="wbot_base_control"/>
     <xacro:wbot_ros2_control
       name="${ros2_control_name}"
